File: schematics/eagle/voltage-amplifier.sch (EAGLE design)
At the start: 15 parts, among them Q1 2N3904, Q2 2N3904, Q3 2N3904, Q4 2N3904

Commit message: Voltage Amplifier PCB
Parts:
- C4, C5, C6: device sym:CAP -> sym-toh:CAP
- Q1, Q2, Q3, Q4: device sym:NPN -> sym-toh:NPN
- R1, R2, R3, R4, R5, R6, R7, R8: device sym:RES -> sym-toh:RES
Connections:
- removed net N$4: R1.A
- removed net N$9: R6.A
- net V+: now also R1.A, R6.A
Other:
- moved on the sheet: R5
Changed lines of the file:
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@@
 <grid distance="0.1" unitdist="inch" unit="inch" style="lines" multiple="1" display="no" altdistance="0.01" altunitdist="inch" altunit="inch"/>
 <layers>
-<layer number="1" name="Top" color="4" fill="1" visible="no" active="no"/>
-<layer number="16" name="Bottom" color="1" fill="1" visible="no" active="no"/>
-<layer number="17" name="Pads" color="2" fill="1" visible="no" active="no"/>
-<layer number="18" name="Vias" color="2" fill="1" visible="no" active="no"/>
-<layer number="19" name="Unrouted" color="6" fill="1" visible="no" active="no"/>
-<layer number="20" name="Dimension" color="24" fill="1" visible="no" active="no"/>
-<layer number="21" name="tPlace" color="7" fill="1" visible="no" active="no"/>
-<layer number="22" name="bPlace" color="7" fill="1" visible="no" active="no"/>
-<layer number="23" name="tOrigins" color="15" fill="1" visible="no" active="no"/>
-<layer number="24" name="bOrigins" color="15" fill="1" visible="no" active="no"/>
-<layer number="25" name="tNames" color="7" fill="1" visible="no" active="no"/>
-<layer number="26" name="bNames" color="7" fill="1" visible="no" active="no"/>
-<layer number="27" name="tValues" color="7" fill="1" visible="no" active="no"/>
-<layer number="28" name="bValues" color="7" fill="1" visible="no" active="no"/>
+<layer number="1" name="Top" color="4" fill="1" visible="yes" active="no"/>
+<layer number="16" name="Bottom" color="1" fill="1" visible="yes" active="no"/>
+<layer number="17" name="Pads" color="2" fill="1" visible="yes" active="no"/>
+<layer number="18" name="Vias" color="2" fill="1" visible="yes" active="no"/>
+<layer number="19" name="Unrouted" color="6" fill="1" visible="yes" active="no"/>
+<layer number="20" name="Dimension" color="24" fill="1" visible="yes" active="no"/>
+<layer number="21" name="tPlace" color="7" fill="1" visible="yes" active="no"/>
+<layer number="22" name="bPlace" color="7" fill="1" visible="yes" active="no"/>
+<layer number="23" name="tOrigins" color="15" fill="1" visible="yes" active="no"/>
+<layer number="24" name="bOrigins" color="15" fill="1" visible="yes" active="no"/>
+<layer number="25" name="tNames" color="7" fill="1" visible="yes" active="no"/>
+<layer number="26" name="bNames" color="7" fill="1" visible="yes" active="no"/>
+<layer number="27" name="tValues" color="7" fill="1" visible="yes" active="no"/>
+<layer number="28" name="bValues" color="7" fill="1" visible="yes" active="no"/>
 <layer number="29" name="tStop" color="7" fill="3" visible="no" active="no"/>
 <layer number="30" name="bStop" color="7" fill="6" visible="no" active="no"/>
@@
 <layer number="35" name="tGlue" color="7" fill="4" visible="no" active="no"/>
 <layer number="36" name="bGlue" color="7" fill="5" visible="no" active="no"/>
-<layer number="37" name="tTest" color="7" fill="1" visible="no" active="no"/>
-<layer number="38" name="bTest" color="7" fill="1" visible="no" active="no"/>
+<layer number="37" name="tTest" color="7" fill="1" visible="yes" active="no"/>
+<layer number="38" name="bTest" color="7" fill="1" visible="yes" active="no"/>
 <layer number="39" name="tKeepout" color="4" fill="11" visible="no" active="no"/>
 <layer number="40" name="bKeepout" color="1" fill="11" visible="no" active="no"/>
@@
 <layer number="44" name="Drills" color="7" fill="1" visible="no" active="no"/>
 <layer number="45" name="Holes" color="7" fill="1" visible="no" active="no"/>
-<layer number="46" name="Milling" color="3" fill="1" visible="no" active="no"/>
-<layer number="47" name="Measures" color="7" fill="1" visible="no" active="no"/>
-<layer number="48" name="Document" color="7" fill="1" visible="no" active="no"/>
-<layer number="49" name="Reference" color="7" fill="1" visible="no" active="no"/>
-<layer number="51" name="tDocu" color="7" fill="1" visible="no" active="no"/>
-<layer number="52" name="bDocu" color="7" fill="1" visible="no" active="no"/>
+<layer number="46" name="Milling" color="3" fill="1" visible="yes" active="no"/>
+<layer number="47" name="Measures" color="7" fill="1" visible="yes" active="no"/>
+<layer number="48" name="Document" color="7" fill="1" visible="yes" active="no"/>
+<layer number="49" name="Reference" color="7" fill="1" visible="yes" active="no"/>
+<layer number="51" name="tDocu" color="7" fill="1" visible="yes" active="no"/>
+<layer number="52" name="bDocu" color="7" fill="1" visible="yes" active="no"/>
 <layer number="88" name="SimResults" color="9" fill="1" visible="no" active="yes"/>
 <layer number="89" name="SimProbes" color="9" fill="1" visible="no" active="yes"/>
@@
 <part name="X_4" library="ngspice-simulation" library_urn="urn:adsk.eagle:library:527439" deviceset="GND" device=""/>
 <part name="X_5" library="ngspice-simulation" library_urn="urn:adsk.eagle:library:527439" deviceset="GND" device=""/>
-<part name="Q2" library="sym" deviceset="NPN" device="" value="2N3904"/>
-<part name="Q3" library="sym" deviceset="NPN" device="" value="2N3904"/>
-<part name="C4" library="sym" deviceset="CAP" device="" value="10u"/>
-<part name="C5" library="sym" deviceset="CAP" device="" value="10u"/>
-<part name="R3" library="sym" deviceset="RES" device="" value="4.7k"/>
-<part name="R6" library="sym" deviceset="RES" device="" value="4.7k"/>
-<part name="R7" library="sym" deviceset="RES" device="" value="100k"/>
-<part name="R8" library="sym" deviceset="RES" device="" value="4.7k"/>
-<part name="C6" library="sym" deviceset="CAP" device="" value="10u"/>
-<part name="Q1" library="sym" deviceset="NPN" device="" value="2N3904"/>
-<part name="R1" library="sym" deviceset="RES" device="" value="4.7k"/>
-<part name="R2" library="sym" deviceset="RES" device="" value="100k"/>
-<part name="Q4" library="sym" deviceset="NPN" device="" value="2N3904"/>
-<part name="R4" library="sym" deviceset="RES" device="" value="4.7k"/>
-<part name="R5" library="sym" deviceset="RES" device="" value="100k"/>
+<part name="Q2" library="sym-toh" deviceset="NPN" device="" value="2N3904"/>
+<part name="Q3" library="sym-toh" deviceset="NPN" device="" value="2N3904"/>
+<part name="C4" library="sym-toh" deviceset="CAP" device="" value="10u"/>
+<part name="C5" library="sym-toh" deviceset="CAP" device="" value="10u"/>
+<part name="R3" library="sym-toh" deviceset="RES" device="" value="4.7k"/>
+<part name="R6" library="sym-toh" deviceset="RES" device="" value="4.7k"/>
+<part name="R7" library="sym-toh" deviceset="RES" device="" value="100k"/>
+<part name="R8" library="sym-toh" deviceset="RES" device="" value="4.7k"/>
+<part name="C6" library="sym-toh" deviceset="CAP" device="" value="10u"/>
+<part name="Q1" library="sym-toh" deviceset="NPN" device="" value="2N3904"/>
+<part name="R1" library="sym-toh" deviceset="RES" device="" value="4.7k"/>
+<part name="R2" library="sym-toh" deviceset="RES" device="" value="100k"/>
+<part name="Q4" library="sym-toh" deviceset="NPN" device="" value="2N3904"/>
+<part name="R4" library="sym-toh" deviceset="RES" device="" value="4.7k"/>
+<part name="R5" library="sym-toh" deviceset="RES" device="" value="100k"/>
 </parts>
 <sheets>
@@
 <attribute name="VALUE" x="290.195" y="15.875" size="1.778" layer="96" align="center-left"/>
 </instance>
-<instance part="R5" gate="G$1" x="279.4" y="2.54" smashed="yes" rot="R270">
-<attribute name="NAME" x="270.51" y="2.54" size="1.778" layer="95" align="bottom-center"/>
-<attribute name="VALUE" x="270.51" y="-2.54" size="1.778" layer="96" align="top-center"/>
+<instance part="R5" gate="G$1" x="271.78" y="2.54" smashed="yes" rot="R270">
+<attribute name="NAME" x="262.89" y="2.54" size="1.778" layer="95" align="bottom-center"/>
+<attribute name="VALUE" x="262.89" y="-2.54" size="1.778" layer="96" align="top-center"/>
 </instance>
 </instances>
@@
 <pinref part="Q4" gate="G$1" pin="B"/>
 <pinref part="R5" gate="G$1" pin="A"/>
+<wire x1="269.24" y1="0" x2="276.86" y2="0" width="0.1524" layer="91"/>
 </segment>
 </net>
@@
 <pinref part="R3" gate="G$1" pin="A"/>
 <wire x1="177.8" y1="22.86" x2="177.8" y2="27.94" width="0.1524" layer="91"/>
-<label x="236.22" y="27.94" size="1.778" layer="95" rot="R90" xref="yes"/>
+<label x="236.22" y="27.686" size="1.778" layer="95" rot="R90" xref="yes"/>
 </segment>
 <segment>
@@
 <segment>
 <label x="152.4" y="27.94" size="1.778" layer="95" rot="R90" xref="yes"/>
+</segment>
+<segment>
+<pinref part="R1" gate="G$1" pin="A"/>
+<wire x1="236.22" y1="25.4" x2="236.22" y2="27.94" width="0.1524" layer="91"/>
+</segment>
+<segment>
+<pinref part="R6" gate="G$1" pin="A"/>
+<wire x1="152.4" y1="22.86" x2="152.4" y2="27.94" width="0.1524" layer="91"/>
 </segment>
 </net>
@@
 <pinref part="Q1" gate="G$1" pin="C"/>
 <wire x1="236.22" y1="7.62" x2="236.22" y2="10.16" width="0.1524" layer="91"/>
-<wire x1="259.08" y1="0" x2="259.08" y2="10.16" width="0.1524" layer="91"/>
-<wire x1="259.08" y1="10.16" x2="236.22" y2="10.16" width="0.1524" layer="91"/>
+<wire x1="251.46" y1="0" x2="251.46" y2="10.16" width="0.1524" layer="91"/>
+<wire x1="251.46" y1="10.16" x2="236.22" y2="10.16" width="0.1524" layer="91"/>
 <junction x="236.22" y="10.16"/>
 <pinref part="R5" gate="G$1" pin="B"/>
-<wire x1="264.16" y1="0" x2="259.08" y2="0" width="0.1524" layer="91"/>
+<wire x1="256.54" y1="0" x2="251.46" y2="0" width="0.1524" layer="91"/>
 </segment>
 </net>
@@
 </segment>
 </net>
-<net name="N$4" class="0">
-<segment>
-<pinref part="R1" gate="G$1" pin="A"/>
-<wire x1="236.22" y1="25.4" x2="236.22" y2="27.94" width="0.1524" layer="91"/>
-</segment>
-</net>
-<net name="N$9" class="0">
-<segment>
-<pinref part="R6" gate="G$1" pin="A"/>
-<wire x1="152.4" y1="22.86" x2="152.4" y2="27.94" width="0.1524" layer="91"/>
-</segment>
-</net>

Commit message: Changed package for the big resistances
Parts:
- R2, R5, R7: device sym-toh:RES -> sym-toh:RES'0309'
Changed lines of the file:
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@@
 <grid distance="0.1" unitdist="inch" unit="inch" style="lines" multiple="1" display="no" altdistance="0.01" altunitdist="inch" altunit="inch"/>
 <layers>
-<layer number="1" name="Top" color="4" fill="1" visible="yes" active="no"/>
-<layer number="16" name="Bottom" color="1" fill="1" visible="yes" active="no"/>
-<layer number="17" name="Pads" color="2" fill="1" visible="yes" active="no"/>
-<layer number="18" name="Vias" color="2" fill="1" visible="yes" active="no"/>
-<layer number="19" name="Unrouted" color="6" fill="1" visible="yes" active="no"/>
-<layer number="20" name="Dimension" color="24" fill="1" visible="yes" active="no"/>
-<layer number="21" name="tPlace" color="7" fill="1" visible="yes" active="no"/>
-<layer number="22" name="bPlace" color="7" fill="1" visible="yes" active="no"/>
-<layer number="23" name="tOrigins" color="15" fill="1" visible="yes" active="no"/>
-<layer number="24" name="bOrigins" color="15" fill="1" visible="yes" active="no"/>
-<layer number="25" name="tNames" color="7" fill="1" visible="yes" active="no"/>
-<layer number="26" name="bNames" color="7" fill="1" visible="yes" active="no"/>
-<layer number="27" name="tValues" color="7" fill="1" visible="yes" active="no"/>
-<layer number="28" name="bValues" color="7" fill="1" visible="yes" active="no"/>
+<layer number="1" name="Top" color="4" fill="1" visible="no" active="no"/>
+<layer number="16" name="Bottom" color="1" fill="1" visible="no" active="no"/>
+<layer number="17" name="Pads" color="2" fill="1" visible="no" active="no"/>
+<layer number="18" name="Vias" color="2" fill="1" visible="no" active="no"/>
+<layer number="19" name="Unrouted" color="6" fill="1" visible="no" active="no"/>
+<layer number="20" name="Dimension" color="24" fill="1" visible="no" active="no"/>
+<layer number="21" name="tPlace" color="7" fill="1" visible="no" active="no"/>
+<layer number="22" name="bPlace" color="7" fill="1" visible="no" active="no"/>
+<layer number="23" name="tOrigins" color="15" fill="1" visible="no" active="no"/>
+<layer number="24" name="bOrigins" color="15" fill="1" visible="no" active="no"/>
+<layer number="25" name="tNames" color="7" fill="1" visible="no" active="no"/>
+<layer number="26" name="bNames" color="7" fill="1" visible="no" active="no"/>
+<layer number="27" name="tValues" color="7" fill="1" visible="no" active="no"/>
+<layer number="28" name="bValues" color="7" fill="1" visible="no" active="no"/>
 <layer number="29" name="tStop" color="7" fill="3" visible="no" active="no"/>
 <layer number="30" name="bStop" color="7" fill="6" visible="no" active="no"/>
@@
 <layer number="35" name="tGlue" color="7" fill="4" visible="no" active="no"/>
 <layer number="36" name="bGlue" color="7" fill="5" visible="no" active="no"/>
-<layer number="37" name="tTest" color="7" fill="1" visible="yes" active="no"/>
-<layer number="38" name="bTest" color="7" fill="1" visible="yes" active="no"/>
+<layer number="37" name="tTest" color="7" fill="1" visible="no" active="no"/>
+<layer number="38" name="bTest" color="7" fill="1" visible="no" active="no"/>
 <layer number="39" name="tKeepout" color="4" fill="11" visible="no" active="no"/>
 <layer number="40" name="bKeepout" color="1" fill="11" visible="no" active="no"/>
@@
 <layer number="44" name="Drills" color="7" fill="1" visible="no" active="no"/>
 <layer number="45" name="Holes" color="7" fill="1" visible="no" active="no"/>
-<layer number="46" name="Milling" color="3" fill="1" visible="yes" active="no"/>
-<layer number="47" name="Measures" color="7" fill="1" visible="yes" active="no"/>
-<layer number="48" name="Document" color="7" fill="1" visible="yes" active="no"/>
-<layer number="49" name="Reference" color="7" fill="1" visible="yes" active="no"/>
-<layer number="51" name="tDocu" color="7" fill="1" visible="yes" active="no"/>
-<layer number="52" name="bDocu" color="7" fill="1" visible="yes" active="no"/>
+<layer number="46" name="Milling" color="3" fill="1" visible="no" active="no"/>
+<layer number="47" name="Measures" color="7" fill="1" visible="no" active="no"/>
+<layer number="48" name="Document" color="7" fill="1" visible="no" active="no"/>
+<layer number="49" name="Reference" color="7" fill="1" visible="no" active="no"/>
+<layer number="51" name="tDocu" color="7" fill="1" visible="no" active="no"/>
+<layer number="52" name="bDocu" color="7" fill="1" visible="no" active="no"/>
 <layer number="88" name="SimResults" color="9" fill="1" visible="no" active="yes"/>
 <layer number="89" name="SimProbes" color="9" fill="1" visible="no" active="yes"/>
@@
 <part name="R3" library="sym-toh" deviceset="RES" device="" value="4.7k"/>
 <part name="R6" library="sym-toh" deviceset="RES" device="" value="4.7k"/>
-<part name="R7" library="sym-toh" deviceset="RES" device="" value="100k"/>
+<part name="R7" library="sym-toh" deviceset="RES" device="'0309'" value="100k"/>
 <part name="R8" library="sym-toh" deviceset="RES" device="" value="4.7k"/>
 <part name="C6" library="sym-toh" deviceset="CAP" device="" value="10u"/>
 <part name="Q1" library="sym-toh" deviceset="NPN" device="" value="2N3904"/>
 <part name="R1" library="sym-toh" deviceset="RES" device="" value="4.7k"/>
-<part name="R2" library="sym-toh" deviceset="RES" device="" value="100k"/>
+<part name="R2" library="sym-toh" deviceset="RES" device="'0309'" value="100k"/>
 <part name="Q4" library="sym-toh" deviceset="NPN" device="" value="2N3904"/>
 <part name="R4" library="sym-toh" deviceset="RES" device="" value="4.7k"/>
-<part name="R5" library="sym-toh" deviceset="RES" device="" value="100k"/>
+<part name="R5" library="sym-toh" deviceset="RES" device="'0309'" value="100k"/>
 </parts>
 <sheets>
